File: smartplug/kicad/sm/sm.sch (KiCad schematic (older format))
At the start: 16 parts, among them J1 Screw_Terminal_01x02, J2 Screw_Terminal_01x02, J4 Screw_Terminal_01x03, T1 HLK-PM01 220-5vDC/3W, T2 HLK-PM03 220-3.3vDC/3W, U1 RELE QC3F-05VDC (10A 125-220 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, U2 ESP8266 ESP-12F

Commit message: freecad
Parts:
- removed C2: Capacitor 22uF, symbol Device:CP1_Small
- removed C4: Capacitor 10uF, symbol Device:CP1_Small
- removed F3: Portafusible para fusible 5x20mm (Quick Blow 630m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, symbol Device:Fuse
- removed F4: Fusible termico 77º, symbol Device:Fuse
- removed T1: HLK-PM01 220-5vDC/3W, Converter_ACDC:Converter_ACDC_Hahn_HS-400xx_THT, symbol Converter_ACDC:HLK-PM01
- removed T2: HLK-PM03 220-3.3vDC/3W, Converter_ACDC:Converter_ACDC_Hahn_HS-400xx_THT, symbol Converter_ACDC:HLK-PM03
- added H1, H2, H3, H4: MountingHole, MountingHole:MountingHole_3.2mm_M3_DIN965, symbol Mechanical:MountingHole
- added J3, J5, J6, J8: Screw_Terminal_01x02, sm:Terminal_Tornillo_2, symbol Connector:Screw_Terminal_01x02
- added J7: Screw_Terminal_01x03, sm:Terminal_Tornillo_3, symbol Connector:Screw_Terminal_01x03
- added J9: Conn_01x06_Male, Connector_PinHeader_1.00mm:PinHeader_1x06_P1.00mm_Vertical, symbol Connector:Conn_01x06_Male
- added R1, R2: Resistencia 200 ohms, Resistor_THT:R_Axial_DIN0204_L3.6mm_D1.6mm_P5.08mm_Horizontal, symbol Device:R
- added U3: Transformador100v-240v_5V_0.6A, sm:Transformador220v-5v, symbol sm-rescue:Transformador100v-240v_5V_0.6A-sm
- C1: footprint (none) -> Connector_PinHeader_1.27mm:PinHeader_1x08_P1.27mm_Vertical
- C3: footprint (none) -> Capacitor_THT:CP_Radial_D5.0mm_P2.50mm
- F1, F2: footprint (none) -> Fuse:Fuseholder_Cylinder-5x20mm_Schurter_0031_8201_Horizontal_Open
- J1, J2: footprint (none) -> sm:Terminal_Tornillo_2
- J4: footprint (none) -> sm:Terminal_Tornillo_3
- RV1: footprint (none) -> Varistor:RV_Disc_D15.5mm_W4.7mm_P7.5mm
- U1: footprint (none) -> sm:Rele_5vDC
- U2: footprint (none) -> sm:ESP8266_ESP-12F3; symbol sm:esp12f -> sm-rescue:esp12f-sm
Connections:
- net labels added: +3.3V, +5V, GND, Linea1, Linea2
- net labels removed: 220v, AC
- wire segments 73 -> 68
Other:
- note added: "(3.3v,5v,GND,D1,Rx,Tx)"
- note added: "Entrada alimentacion 220V"
- note added: "Fusible termico 77º"
- note added: "Led Rojo (+ -)"
- note added: "Led Verde (+ -)"
- note added: "Pines para futuras aplicaciones"
- note added: "Rele (- señal +)"
- note added: "Rele (Open Middle)"
- note added: "Salida (L1 L2)"
- note added: "Sensor Movimiento (- Señal +)"
- moved on the sheet: C1, C3, F1, F2, J1, J2, RV1, U1, U2
