File: PhotoPlug/kicad/PhotoPlug/PhotoPlug.kicad_pcb (KiCad board)
At the start: 2 copper layers, 20 parts, among them IC1 ESP32-CAM, J1 Screw_Terminal_01x02, J2 Screw_Terminal_01x03, J3 Screw_Terminal_01x02, J4 Conn_01x08_MountingPin, J5 Screw_Terminal_01x02, K1 SRD-05VDC-SL-C, U2 Transformador100v-240v_5V_0.6A

Commit message: CajaLimpia
Parts:
- removed D1, D2, D3: LED, LED_THT:LED_D3.0mm
- removed REF**: MountingHole_3.2mm_M3_DIN965, MountingHole:MountingHole_3.2mm_M3_DIN965
- removed U2: Transformador100v-240v_5V_0.6A, PhotoPlug:TSP-05
- added H1: MountingHole, MountingHole:MountingHole_3.5mm, F.Cu at (119.1, 99.3)
- added H2: MountingHole, MountingHole:MountingHole_3.5mm, F.Cu at (118.6, 151.4)
- added H3: MountingHole, MountingHole:MountingHole_3.5mm, F.Cu at (201.2, 99.1)
- added H4: MountingHole, MountingHole:MountingHole_3.5mm, F.Cu at (201.2, 151.1)
- added J6: Conn_01x02_MountingPin, Connector_PinHeader_1.00mm:PinHeader_1x02_P1.00mm_Vertical, F.Cu at (201.2, 124.5)
- added J7: Conn_01x02_MountingPin, Connector_PinHeader_1.00mm:PinHeader_1x02_P1.00mm_Vertical, F.Cu at (200.9, 130.3)
- added J8: Conn_01x02_MountingPin, Connector_PinHeader_1.00mm:PinHeader_1x02_P1.00mm_Vertical, F.Cu at (201.4, 120.1)
- added U1: Transformador100v-240v_5V_0.6A, milib:Transformador Tenstar Robot, F.Cu at (126.2, 127.0)
- F1, F2: footprint Fuse:Fuseholder_Blade_Mini_Keystone_3568 -> milib:MiFusible
- J1, J3, J5: footprint TerminalBlock_Altech:Altech_AK300_1x02_P5.00mm_45-Degree -> milib:Altech_AK300_1x02_P5.00mm_45-Degree
- J2: footprint TerminalBlock_Altech:Altech_AK300_1x03_P5.00mm_45-Degree -> milib:Altech_AK300_1x03_P5.00mm_45-Degree
- J4: footprint Connector_PinSocket_1.00mm:PinSocket_1x08_P1.00mm_Vertical_SMD_Pin1Left -> Connector_PinSocket_1.00mm:PinSocket_1x08_P1.00mm_Vertical
- RV1: footprint Varistor:RV_Disc_D12mm_W4.8mm_P7.5mm -> milib:RV_Disc_D12mm_W4.8mm_P7.5mm
- moved J1 163.8 mm to (196.6, 138.7), turned to 0 degrees
- moved J3 138.8 mm to (186.7, 109.0), turned to 0 degrees
- moved J2 132.7 mm to (176.0, 147.1), turned to 0 degrees
- moved R1 118.1 mm to (196.1, 129.5)
- moved C2 118.0 mm to (186.7, 132.6), turned to 0 degrees
- moved R3 117.3 mm to (195.6, 125.0), turned to 180 degrees
- moved R2 116.6 mm to (195.3, 120.7)
- moved C1 115.1 mm to (186.2, 121.2), turned to 0 degrees
- moved RV1 102.0 mm to (142.7, 110.0), turned to 90 degrees
- moved F1 99.6 mm to (158.2, 147.1), turned to 0 degrees
- moved F2 86.6 mm to (134.6, 149.4), turned to 180 degrees
- moved J4 64.6 mm to (150.1, 115.1), turned to 180 degrees
- moved K1 58.6 mm to (145.5, 135.9), turned to 90 degrees
- moved IC1 40.1 mm to (156.7, 120.4), turned to 0 degrees
- moved J5 33.6 mm to (130.8, 105.4)
Routing:
- net Net-(J1-Pad2): track 0.00 -> 176.4 mm, vias 0 -> 2
- net GND: track 0.00 -> 116.6 mm, vias 0 -> 2
- net Net-(F1-Pad2): track 0.00 -> 79.3 mm
- net Net-(J2-Pad1): track 0.00 -> 73.7 mm
- net Net-(IC1-Pad4): track 0.00 -> 70.5 mm
- net +1V5: track 0.00 -> 64.4 mm
- net Net-(J1-Pad1): track 0.00 -> 59.5 mm
- net Net-(IC1-Pad6): track 0.00 -> 48.4 mm
- net Net-(F2-Pad2): track 0.00 -> 40.4 mm
- net Net-(F1-Pad1): track 0.00 -> 34.3 mm
- net Net-(IC1-Pad1): track 0.00 -> 13.1 mm
- net +5V: track 0.00 -> 12.5 mm
- net Net-(IC1-Pad2): track 0.00 -> 11.6 mm
- net Net-(IC1-Pad3): track 0.00 -> 10.1 mm
- net Net-(J8-Pad2): track 0.00 -> 6.72 mm
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Other:
- board outline added: 90.2 x 59.9 mm
- board text added: "PELIGRO 220V"
